File: Electronics/7_segment_display/7_segment_display.kicad_sch (KiCad schematic)
At the start: 18 parts, among them J1 AVR ISP, SW1 Reset, U1 ATMEGA328P-PU, U2 SH5461AS, Y1 16 MHz

Commit message: PCB for testing(home made)
Parts:
- removed SW1: Reset, symbol Switch:SW_MEC_5E
- added SW1: Reset, Button_Switch_THT:SW_PUSH_6mm_H5mm, symbol Switch:SW_Push_Dual_x2
- C1, C2: footprint (none) -> Capacitor_THT:C_Disc_D3.0mm_W1.6mm_P2.50mm
- C3: footprint (none) -> Capacitor_THT:CP_Radial_D4.0mm_P1.50mm
- J1: footprint (none) -> Connector_PinHeader_2.54mm:PinHeader_2x03_P2.54mm_Vertical
- R1, R10, R2, R3, R4, R5, R6, R7, R8, R9: footprint (none) -> Resistor_THT:R_Axial_DIN0207_L6.3mm_D2.5mm_P7.62mm_Horizontal
- Y1: footprint (none) -> Crystal:Crystal_HC49-4H_Vertical
Connections:
- net GND: now also SW1.1 (C)
- net Reset: now also SW1.2 (D)
